Commit message: edit tb3 move

File: tb3_description/turtlebot3_waffle.urdf.xacro (robot description, xacro)
@@ -62,5 +62,5 @@
                iyy="1.1192413e-05" iyz="-1.4400107e-11"
                izz="2.0712558e-05" />
-      </inertial>
+    </inertial>
   </link>
   <joint name="wheel_right_joint" type="continuous">
@@ -90,5 +90,5 @@
                iyy="1.1192413e-05" iyz="-1.4400107e-11"
                izz="2.0712558e-05" />
-      </inertial>
+    </inertial>
   </link>
   <joint name="caster_back_right_joint" type="fixed">
@@ -219,5 +219,5 @@
   <joint name="camera_joint_dang" type="fixed">
     <axis xyz="0 1 0" />
-    <origin xyz="0 0 0.12" rpy="0 0 0"/>
+    <origin xyz="-0.18 0 0.12" rpy="0 0 3.141592"/>
     <parent link="base_link"/>
     <child link="camera_link_dang"/>
@@ -226,5 +226,5 @@
   <link name="camera_link_dang">
     <collision>
-      <origin xyz="0 0 0" rpy="0 0 0"/>
+      <origin xyz="0 0 0" rpy="0 0 3.141592"/>
       <geometry>
         <box size="${camera_link} ${camera_link} ${camera_link}"/>
@@ -232,5 +232,5 @@
     </collision>
     <visual>
-      <origin xyz="0 0 0" rpy="0 0 0"/>
+      <origin xyz="0 0 0" rpy="0 0 3.141592"/>
       <geometry>
         <box size="${camera_link} ${camera_link} ${camera_link}"/>
@@ -239,5 +239,5 @@
     <inertial>
       <mass value="1e-5" />
-      <origin xyz="0 0 0" rpy="0 0 0"/>
+      <origin xyz="0 0 0" rpy="0 0 3.141592"/>
       <inertia ixx="1e-6" ixy="0" ixz="0" iyy="1e-6" iyz="0" izz="1e-6" />
     </inertial>
